Commit message: modified comments and indentation.

File: urdf/robot_description.urdf.xacro (robot description, xacro)
@@ -6,25 +6,18 @@
   xmlns:xacro="http://ros.org/wiki/xacro"
   name="robot_description">
-<!-- inertial measurement unit for gazebo -->
+<!-- IMU -->
 <xacro:include filename="$(find uos_common_urdf)/urdf/imu.gazebo.urdf.xacro" />
 <xacro:property name="imu_stdev" value="0.00017" />
 <xacro:imu_gazebo link="base_link" imu_topic="imu" update_rate="100.0" stdev="${imu_stdev}" />
- <!--link name="imu" />
-  <joint name="base_link_to_imu_joint" type="fixed">
-    <parent link="base_link" />
-    <child link="imu" />
-    <origin xyz="0 0 0" rpy="0 0 0" />
-  </joint-->
-<!-- Laser_scan -->
+<!-- Laserscanner LMS1xx -->
 <xacro:include filename="$(find uos_common_urdf)/urdf/sick_lms100.urdf.xacro" />
 <xacro:sick_lms100 laser_link="laser" gazebo_topic="scan" />
-<!--link name="laser_scan" /-->
 <joint name="laser_scan_joint" type="fixed">
-    <origin xyz="0.07 0 0.025" rpy="-3.14 0 0" />
-    <parent link="front_surface"/>
-    <child link="laser" />
-  </joint>
-  <!-- base_footprint is a fictitious link(frame) that is on the ground right below base_link origin,
-       navigation stack depends on this frame -->
+  <origin xyz="0.07 0 0.025" rpy="-3.14 0 0" />
+  <parent link="front_surface"/>
+  <child link="laser" />
+</joint>
+<!-- base_footprint is a imaginary link(frame) that is on the ground directly below base_link origin,
+	navigation stack depends on this frame. It makes the robot load on the base plane instead of inside it. -->
   <link name="base_footprint"/>
   <joint name="base_footprint_joint" type="fixed">
@@ -33,5 +26,5 @@
     <parent link="base_footprint" />
   </joint>
-<!--Box_Links -->
+<!--Box_Links. They build the frame of the robot. -->
 <xacro:macro name="robot_box" params="name size xyz rpy inertial_mass gazebo_color" >
     <link name="${name}">
@@ -52,10 +45,10 @@
         </collision>
       <inertial>
-      <mass value="${inertial_mass}"/>
+        <mass value="${inertial_mass}"/>
         <origin xyz="0 0 0" />
         <inertia ixx="0.00000001" ixy="0.0" ixz="0.0"
                  iyy="0.00000001" iyz="0.0"
                  izz="0.00000001" />
-    </inertial>
+	  </inertial>
     </link>
   <gazebo reference="${name}">
@@ -68,5 +61,5 @@
 <xacro:robot_box name="front_surface" size="0.02 0.29 0.14" xyz="0 0 0" rpy="0 0 0" inertial_mass="0.5" gazebo_color="Gazebo/Grey"/>
 <xacro:robot_box name="back_surface"  size="0.02 0.43 0.08" xyz="0 0 0" rpy="0 0 0" inertial_mass="0.5" gazebo_color="Gazebo/Grey"/>
-<!-- Box_joints -->
+<!-- Box_joints. These link the parts of the frame-->
 <xacro:macro name="bjoint" params="type child xyz rpy">
    <joint name=" ${child}_joint" type= "${type}" >
@@ -80,5 +73,5 @@
 <xacro:bjoint type="fixed" child="front_surface" xyz="0.205 0 -0.03" rpy="0 0 0"/>
 <xacro:bjoint type="fixed" child="back_surface" xyz="-0.205 0 0" rpy="0 0 0"/>
-<!--Cylinder_links (front_wheels & base_for_back_wheels)     ojo:falta la mass!-->
+<!--Cylinder_links. front cylinders are the wheels and rotate. back cylindars are fixed and are attached to the caster-ball wheels -->
 <xacro:macro name="robot_cylinder" params="name length radius rpy material inertial_mass rgba gazebo_color">
 <link name="${name}">
@@ -99,11 +92,11 @@
         </collision>
     <inertial>
-   <mass value="${inertial_mass}" />
+      <mass value="${inertial_mass}" />
         <origin xyz="0 0 0" />
         <inertia ixx="0.001" ixy="0.0" ixz="0.0"
                  iyy="0.001" iyz="0.0"
                  izz="0.001" />
-</inertial>
- </link>
+    </inertial>
+</link>
   <gazebo reference="${name}">
    <material value="${gazebo_color}"/>
@@ -139,5 +132,5 @@
 <xacro:cjoint axis="0 0 0" type="fixed" parent="base_link" child="back_left_wheel_base" xyz="-0.1405 0.11 -0.06" rpy="0 0 0"/>
 <xacro:cjoint axis="0 0 0" type="fixed" parent="base_link" child="back_right_wheel_base" xyz="-0.1405 -0.11 -0.06" rpy="0 0 0"/>
-<!-- Sphere_Links (Back_wheels) -->
+<!-- Sphere_Links (Back_wheels). The actual robot has caster wheels because they're cheaper. The simulation has caster ball wheels because they're easier to model.-->
 <xacro:macro name="robot_sphere" params="name radius xyz rpy">
     <link name="${name}">
@@ -164,5 +157,5 @@
       </inertial>
 </link>
- <!-- friction parameters -->
+ <!-- friction parameters. -->
   <gazebo reference="${name}">
     <mu1>1.0</mu1>
@@ -177,5 +170,5 @@
 <xacro:robot_sphere name="left_back_wheel" radius="0.035" xyz="0 0 0" rpy="0 0 0"/>
 <xacro:robot_sphere name="right_back_wheel" radius="0.035" xyz="0 0 0" rpy="0 0 0" />
-<!-- Sphere_joints -->
+<!-- Sphere_joints. Must be continuous for the caster wheels to freely spin. -->
 <xacro:macro name="sjoint" params="axis type parent child xyz rpy">
    <axis xyz="${axis}"/>
@@ -192,4 +185,5 @@
 <xacro:sjoint axis="0 1 0" type="continuous" parent="back_right_wheel_base" child="right_back_wheel" xyz="0 0 -0.0525"
 rpy="0 0 0" />
+<!-- defines the robot joint state so teleop commands can make the robot move. -->
 <gazebo>
     <plugin name="robot_description" filename="libgazebo_ros_diffdrive_uos.so">
@@ -199,7 +193,5 @@
       <joint_states_topic_name>joint_states</joint_states_topic_name>
       <left_front_wheel_joint>left_front_wheel_joint</left_front_wheel_joint>
-      <!--left_rear_wheel_joint>left_front_wheel_joint</left_rear_wheel_joint-->
       <right_front_wheel_joint>right_front_wheel_joint</right_front_wheel_joint>
-      <!--right_rear_wheel_joint>right_front_wheel_joint</right_rear_wheel_joint-->
       <wheel_separation>0.30</wheel_separation>
       <wheel_diameter>0.18</wheel_diameter>
@@ -210,5 +202,5 @@
     </plugin>
   </gazebo>
-  <!-- publish ground truth for pose of base_footprint -->
+<!-- publish ground truth for pose of base_footprint -->
 <gazebo>
     <plugin name="base_footprint_controller" filename="libgazebo_ros_p3d.so">
